File: PCBv2/PCBv2/PCBv2.kicad_pcb (KiCad board)
At the start: 2 copper layers, 20 parts, among them J1 USB_C_Receptacle_USB2.0, SW1 SW_SPST, SW2 SW_SPDT, U1 ATtiny412-SS, U2 MCP73831-2-OT

Commit message: v2 Updates, not tested yet
Parts:
- BT1: moved to B.Cu
- SW1, SW2: moved to F.Cu
- moved D1 96.8 mm to (150.0, 56.0)
- moved D5 63.3 mm to (68.0, 56.0)
- moved D2 58.2 mm to (131.0, 56.0)
- moved D4 39.1 mm to (86.0, 56.0)
- moved D3 35.8 mm to (109.0, 56.0)
- moved R3 18.9 mm to (65.0, 48.0), turned to 90 degrees
- moved R4 17.5 mm to (150.0, 48.8), turned to -90 degrees
- moved R2 14.4 mm to (68.8, 53.0), turned to 90 degrees
- moved C1 13.1 mm to (150.0, 53.2), turned to -90 degrees
- moved C2 11.0 mm to (68.8, 59.0), turned to 90 degrees
- moved R1 9.25 mm to (68.2, 48.0), turned to 90 degrees
- moved R5 7.21 mm to (150.0, 58.8), turned to -90 degrees
- moved J1 5.50 mm to (61.5, 56.0)
- moved SW2 4.95 mm to (69.8, 47.2), turned to 180 degrees
- moved U1 4.10 mm to (155.8, 56.0), turned to 90 degrees
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Routing:
- net /CHGSTAT: track 0.00 -> 107.0 mm
- net +BATT: track 0.00 -> 41.2 mm, vias 0 -> 7
- net Earth: track 0.00 -> 29.9 mm, vias 0 -> 5
- net Net-(BT1-Pad1): track 0.00 -> 22.7 mm
- net Net-(D3-Pad2): track 0.00 -> 19.4 mm
- net +5V: track 0.00 -> 18.7 mm, vias 0 -> 2
- net Net-(D2-Pad2): track 0.00 -> 18.4 mm
- net Net-(R3-Pad1): track 0.00 -> 17.7 mm
- net Net-(D4-Pad2): track 0.00 -> 16.3 mm, vias 0 -> 2
- net Net-(D1-Pad2): track 0.00 -> 16.2 mm
- net Net-(SW1-Pad1): track 0.00 -> 11.0 mm, vias 0 -> 1
- net /BATSTAT: track 0.00 -> 10.9 mm
- net Net-(J1-PadB5): track 0.00 -> 7.01 mm
- net Net-(J1-PadA5): track 0.00 -> 5.74 mm
- net Net-(D1-Pad4): track 0.00 -> 5.29 mm, vias 0 -> 1
- added copper zone on B.Cu, net +BATT
- added copper zone on F.Cu, net Earth
Other:
- board outline added: 100 x 22 mm
